File: arisu.kicad_pcb (KiCad board)
At the start: 2 copper layers, 339.1 x 118.7 mm, 176 parts, among them J1 USB_B_Micro, SW1 SW_Push, SW10 SW_Push, SW11 SW_Push, SW12 SW_Push, SW13 SW_Push, SW14 SW_Push, SW15 SW_Push, SW16 SW_Push, SW17 SW_Push, SW18 SW_Push, SW19 SW_Push, SW2 SW_Push, SW20 SW_Push, SW21 SW_Push, SW22 SW_Push, SW23 SW_Push, SW24 SW_Push, SW25 SW_Push, SW26 SW_Push, SW27 SW_Push, SW28 SW_Push, SW29 SW_Push, SW3 SW_Push, SW30 SW_Push, SW31 SW_Push, SW32 SW_Push, SW33 SW_Push, SW34 SW_Push, SW35 SW_Push, SW36 SW_Push, SW37 SW_Push, SW38 SW_Push, SW39 SW_Push, SW4 SW_Push, SW40 SW_Push, SW41 SW_Push, SW42 SW_Push, SW43 SW_Push, SW44 SW_Push, SW45 SW_Push, SW46 SW_Push, SW47 SW_Push, SW48 SW_Push, SW49 SW_Push, SW5 SW_Push, SW50 SW_Push, SW51 SW_Push, SW52 SW_Push, SW53 SW_Push, SW54 SW_Push, SW55 SW_Push, SW56 SW_Push, SW57 SW_Push, SW58 SW_Push, SW59 SW_Push, SW6 SW_Push, SW60 SW_Push, SW61 SW_Push, SW62 SW_Push, SW63 SW_Push, SW64 SW_Push, SW65 SW_Push, SW66 SW_Push, SW67 SW_Push, SW7 SW_Push, SW8 SW_Push, SW9 SW_Push, U1 USBLC6-2SC6, U2 ATmega32U4-AU, Y1 Crystal_GND24

Commit message: changed files to have type c and updated gerber
Parts:
- removed J1: USB_B_Micro, Connectors_USB:USB_Micro-B_Molex-105017-0001
- added R5: 5.1k, Resistor_SMD:R_0805_2012Metric_Pad1.20x1.40mm_HandSolder, B.Cu at (169.5, 30.0)
- added R6: 5.1k, Resistor_SMD:R_0805_2012Metric_Pad1.20x1.40mm_HandSolder, B.Cu at (182.5, 26.5)
- added USB1: HRO-TYPE-C-31-M-12, Type-C:HRO-TYPE-C-31-M-12, B.Cu at (175.5, 23.5)
- moved U1 1.16 mm to (166.0, 29.5)
- moved C4 0.40 mm to (181.5, 30.2)
- moved C3 0.37 mm to (183.5, 30.2)
- renumbered PF6 to J10, PF7 to J11, VCC to J12, D+ to J13, D- to J14, GND to J15, MISO to J2, VCC to J3, SCK to J4, MOSI to J5, RES to J6, GND to J7, PF4 to J8, PF5 to J9
Connections:
- net /~RES~ renamed /~{RES}
- U1 pad 1: Net-(U1-Pad1) -> unconnected-(U1-Pad1)
- U1 pad 3: Net-(U1-Pad3) -> unconnected-(U1-Pad3)
- U2 pad 42: Net-(U2-Pad42) -> unconnected-(U2-Pad42)
Routing:
- net GND: track 71.6 -> 101.4 mm, vias 12 -> 11
- net VCC: track 205.4 -> 213.3 mm, vias 9 -> 11
- net Net-(J14-Pad1): track 45.1 -> 37.7 mm
- net Net-(R6-Pad2): track 0.00 -> 6.95 mm
- net Net-(R5-Pad2): track 0.00 -> 6.51 mm
- net Net-(J13-Pad1): track 47.8 -> 53.4 mm
- net /row0: track 328.0 -> 327.3 mm
Other:
- net class Default removed
- net class Power removed
